Commit message: Sensores acivos y gazebo funcional

File: src/marvin_description/urdf/controller/ackermann_drive.xacro (robot description, xacro)
@@ -1,12 +1,12 @@
+<?xml version="1.0"?>
 <robot xmlns:xacro="http://ros.org/wiki/xacro">
-    <xacro:macro name="ackermann_drive_controller">
         <gazebo>
             <plugin name="differential_drive_controller" filename="libgazebo_ros_diff_drive.so">
                 <ros>
                     <!-- <namespace></namespace> -->
-                    <remapping>cmd_vel:=cmd_vel</remapping>
                     <remapping>odom:=odom/unfiltered</remapping>
                 </ros>
                 <updateRate>100</updateRate>
+                <!-- Wheel Information -->
                 <num_wheel_pairs>2</num_wheel_pairs>
                 <left_joint>joint_back_wheel_left</left_joint>
@@ -16,17 +16,15 @@
                 <wheel_separation>0.154</wheel_separation>
                 <wheel_diameter>0.0635</wheel_diameter>
+                <!-- Limits -->
+                <max_wheel_torque>2.4</max_wheel_torque>
                 <max_wheel_acceleration>5.0</max_wheel_acceleration>
-                <max_wheel_torque>2.4</max_wheel_torque>
+                <!-- Output -->
+                <odometry_frame>odom</odometry_frame>
                 <robot_base_frame>base_footprint</robot_base_frame>
-                <commandTopic>cmd_vel</commandTopic>
-                <odometryTopic>odom</odometryTopic>
                 <publish_odom>true</publish_odom>
+                <publish_odom_tf>true</publish_odom_tf>
+                <publish_wheel_tf>true</publish_wheel_tf>
                 <odometry_source>1</odometry_source>
-                <publish_odom_tf>false</publish_odom_tf>
-                <publish_wheel_tf>true</publish_wheel_tf>
-                <odometry_frame>odom</odometry_frame>
-                <legacyMode>false</legacyMode>
             </plugin>
         </gazebo>
-    </xacro:macro>
 </robot>

File: src/marvin_description/urdf/marvin.urdf.xacro (robot description, xacro)
@@ -5,9 +5,10 @@
      For more information, please see http://wiki.ros.org/sw_urdf_exporter -->
 <robot name="vehicle_model" xmlns:xacro="http://ros.org/wiki/xacro">
-    <xacro:include filename="$(find marvin_description)/urdf/sensors/depth_camera.urdf.xacro" />
-    <xacro:include filename="$(find marvin_description)/urdf/sensors/imu.urdf.xacro" />
-    <xacro:include filename="$(find marvin_description)/urdf/sensors/lidar.urdf.xacro" />
-    <xacro:include
-        filename="$(find marvin_description)/urdf/controller/ackermann_drive.urdf.xacro" />
+    <xacro:include filename="$(find marvin_description)/urdf/controller/ackermann_drive.xacro" />
+    <xacro:include filename="$(find marvin_description)/urdf/sensors/imu.xacro" />
+    <xacro:include filename="$(find marvin_description)/urdf/sensors/lidar.xacro" />
+    <xacro:include filename="$(find marvin_description)/urdf/sensors/camera_right.xacro" />
+    <xacro:include filename="$(find marvin_description)/urdf/sensors/camera_left.xacro" />
+    <xacro:include filename="$(find marvin_description)/urdf/sensors/camera_depth.xacro" />
     <link
         name="base_link">
@@ -208,5 +209,5 @@
     <joint
         name="joint_front_handle_left"
-        type="revolute">
+        type="fixed">
         <origin
             xyz="0.13072 0.057509 -0.010582"
@@ -326,5 +327,5 @@
     <joint
         name="joint_front_handle_right"
-        type="revolute">
+        type="fixed">
         <origin
             xyz="0.13072 -0.055491 -0.010582"
@@ -402,110 +403,4 @@
             friction="0.1" />
     </joint>
-    <link
-        name="camera_left">
-        <inertial>
-            <origin
-                xyz="1.3517E-07 -0.00025619 0.0067093"
-                rpy="0 0 0" />
-            <mass
-                value="0.0050148" />
-            <inertia
-                ixx="3.1349E-07"
-                ixy="3.05E-12"
-                ixz="-9.2173E-12"
-                iyy="3.4979E-07"
-                iyz="-3.6215E-11"
-                izz="2.6383E-07" />
-        </inertial>
-        <visual>
-            <origin
-                xyz="0 0 0"
-                rpy="0 0 0" />
-            <geometry>
-                <mesh
-                    filename="package://marvin_description/meshes/camera_left.STL" />
-            </geometry>
-            <material
-                name="">
-                <color
-                    rgba="0.25098 0.25098 0.25098 1" />
-            </material>
-        </visual>
-        <collision>
-            <origin
-                xyz="0 0 0"
-                rpy="0 0 0" />
-            <geometry>
-                <mesh
-                    filename="package://marvin_description/meshes/camera_left.STL" />
-            </geometry>
-        </collision>
-    </link>
-    <joint
-        name="joint_camera_left"
-        type="fixed">
-        <origin
-            xyz="-0.005 0.048531 0.095"
-            rpy="0 0 0" />
-        <parent
-            link="base_link" />
-        <child
-            link="camera_left" />
-        <axis
-            xyz="0 0 0" />
-    </joint>
-    <link
-        name="camera_right">
-        <inertial>
-            <origin
-                xyz="1.361E-07 -0.00025619 0.0067093"
-                rpy="0 0 0" />
-            <mass
-                value="0.0050148" />
-            <inertia
-                ixx="3.1349E-07"
-                ixy="3.0256E-12"
-                ixz="-9.2702E-12"
-                iyy="3.4979E-07"
-                iyz="-3.6066E-11"
-                izz="2.6383E-07" />
-        </inertial>
-        <visual>
-            <origin
-                xyz="0 0 0"
-                rpy="0 0 0" />
-            <geometry>
-                <mesh
-                    filename="package://marvin_description/meshes/camera_right.STL" />
-            </geometry>
-            <material
-                name="">
-                <color
-                    rgba="0.25098 0.25098 0.25098 1" />
-            </material>
-        </visual>
-        <collision>
-            <origin
-                xyz="0 0 0"
-                rpy="0 0 0" />
-            <geometry>
-                <mesh
-                    filename="package://marvin_description/meshes/camera_right.STL" />
-            </geometry>
-        </collision>
-    </link>
-    <joint
-        name="joint_camera_right"
-        type="fixed">
-        <origin
-            xyz="-0.005 -0.048531 0.095"
-            rpy="0 0 0" />
-        <parent
-            link="base_link" />
-        <child
-            link="camera_right" />
-        <axis
-            xyz="0 0 0" />
-    </joint>
     <!-- Robot Footprint -->
     <link name="base_footprint" />
@@ -564,5 +459,4 @@
         <material>Gazebo/White</material>
     </gazebo>
-    <xacro:imu />
     <xacro:lidar
         update_rate="10"
@@ -575,5 +469,3 @@
         topic_name="base/scan">
     </xacro:lidar>
-    <xacro:depth_camera />
-    <xacro:ackermann_drive_controller />
 </robot>

File: src/marvin_description/urdf/sensors/imu.xacro (robot description, xacro)
@@ -1,4 +1,4 @@
+<?xml version="1.0"?>
 <robot xmlns:xacro="http://ros.org/wiki/xacro">
-    <xacro:macro name="imu">
       <link name="imu_link"/>
       <joint name="imu_to_base_link" type="fixed">
@@ -30,4 +30,3 @@
         </sensor>
       </gazebo>
-    </xacro:macro>
   </robot>

File: src/marvin_description/urdf/sensors/lidar.xacro (robot description, xacro)
@@ -1,2 +1,3 @@
+<?xml version="1.0"?>
 <robot xmlns:xacro="http://ros.org/wiki/xacro">
     <xacro:property name="M_PI" value="3.1415926535897931" />
