Commit message: Mapeo y localizacoin refinadas

File: src/marvin_description/urdf/marvin.urdf.xacro (robot description, xacro)
@@ -29,5 +29,5 @@
         <visual>
             <origin
-                xyz="0 0 0"
+                xyz="0 0 0.02"
                 rpy="0 0 0" />
             <geometry>
@@ -403,12 +403,11 @@
             friction="0.1" />
     </joint>
-    <!-- Robot Footprint
+    <!-- Robot Footprint -->
     <link name="base_footprint" />
     <joint name="base_joint" type="fixed">
-        <parent link="base_footprint" />
-        <child link="base_link" />
-        <origin xyz="0 0 0.06" rpy="0 0 0" />
-    </joint>
--->
+        <parent link="base_link" />
+        <child link="base_footprint" />
+        <origin xyz="0 0 0" rpy="0 0 0" />
+    </joint>
     <gazebo reference="base_link">
         <mu1>200</mu1>
