Commit message: wrwerwe

File: marvin_sim_ws/src/marvin_description/urdf/controller/ackermann_drive.xacro (robot description, xacro)
@@ -21,5 +21,5 @@
                 <!-- Output -->
                 <odometry_frame>odom</odometry_frame>
-                <robot_base_frame>base_link</robot_base_frame>
+                <robot_base_frame>base_footprint</robot_base_frame>
                 <publish_odom>true</publish_odom>
                 <publish_odom_tf>true</publish_odom_tf>

File: marvin_sim_ws/src/marvin_description/urdf/marvin.urdf.xacro (robot description, xacro)
@@ -5,10 +5,10 @@
      For more information, please see http://wiki.ros.org/sw_urdf_exporter -->
 <robot name="vehicle_model" xmlns:xacro="http://ros.org/wiki/xacro">
-    <xacro:include filename="$(find marvincar_description)/urdf/controller/ackermann_drive.xacro" />
-    <xacro:include filename="$(find marvincar_description)/urdf/sensors/imu.xacro" />
-    <xacro:include filename="$(find marvincar_description)/urdf/sensors/lidar.xacro" />
-    <xacro:include filename="$(find marvincar_description)/urdf/sensors/camera_right.xacro" />
-    <xacro:include filename="$(find marvincar_description)/urdf/sensors/camera_left.xacro" />
-    <xacro:include filename="$(find marvincar_description)/urdf/sensors/camera_depth.xacro" />
+    <xacro:include filename="$(find marvin_description)/urdf/controller/ackermann_drive.xacro" />
+    <xacro:include filename="$(find marvin_description)/urdf/sensors/imu.xacro" />
+    <xacro:include filename="$(find marvin_description)/urdf/sensors/lidar.xacro" />
+    <xacro:include filename="$(find marvin_description)/urdf/sensors/camera_right.xacro" />
+    <xacro:include filename="$(find marvin_description)/urdf/sensors/camera_left.xacro" />
+    <xacro:include filename="$(find marvin_description)/urdf/sensors/camera_depth.xacro" />
     <link
         name="base_link">
@@ -33,5 +33,5 @@
             <geometry>
                 <mesh
-                    filename="package://marvincar_description/meshes/base_link.STL" />
+                    filename="package://marvin_description/meshes/base_link.STL" />
             </geometry>
             <material
@@ -47,5 +47,5 @@
             <geometry>
                 <mesh
-                    filename="package://marvincar_description/meshes/base_link.STL" />
+                    filename="package://marvin_description/meshes/base_link.STL" />
             </geometry>
         </collision>
@@ -73,19 +73,19 @@
             <geometry>
                 <mesh
-                    filename="package://marvincar_description/meshes/back_wheel_left.STL" />
-            </geometry>
-            <material
-                name="">
-                <color
-                    rgba="0.79216 0.81961 0.93333 1" />
-            </material>
-        </visual>
-        <collision>
-            <origin
-                xyz="0 0 0"
-                rpy="0 0 0" />
-            <geometry>
-                <mesh
-                    filename="package://marvincar_description/meshes/back_wheel_left.STL" />
+                    filename="package://marvin_description/meshes/back_wheel_left.STL" />
+            </geometry>
+            <material
+                name="">
+                <color
+                    rgba="0.79216 0.81961 0.93333 1" />
+            </material>
+        </visual>
+        <collision>
+            <origin
+                xyz="0 0 0"
+                rpy="0 0 0" />
+            <geometry>
+                <mesh
+                    filename="package://marvin_description/meshes/back_wheel_left.STL" />
             </geometry>
         </collision>
@@ -131,19 +131,19 @@
             <geometry>
                 <mesh
-                    filename="package://marvincar_description/meshes/back_wheel_right.STL" />
-            </geometry>
-            <material
-                name="">
-                <color
-                    rgba="0.79216 0.81961 0.93333 1" />
-            </material>
-        </visual>
-        <collision>
-            <origin
-                xyz="0 0 0"
-                rpy="0 0 0" />
-            <geometry>
-                <mesh
-                    filename="package://marvincar_description/meshes/back_wheel_right.STL" />
+                    filename="package://marvin_description/meshes/back_wheel_right.STL" />
+            </geometry>
+            <material
+                name="">
+                <color
+                    rgba="0.79216 0.81961 0.93333 1" />
+            </material>
+        </visual>
+        <collision>
+            <origin
+                xyz="0 0 0"
+                rpy="0 0 0" />
+            <geometry>
+                <mesh
+                    filename="package://marvin_description/meshes/back_wheel_right.STL" />
             </geometry>
         </collision>
@@ -189,19 +189,19 @@
             <geometry>
                 <mesh
-                    filename="package://marvincar_description/meshes/front_handle_left.STL" />
-            </geometry>
-            <material
-                name="">
-                <color
-                    rgba="0.79216 0.81961 0.93333 1" />
-            </material>
-        </visual>
-        <collision>
-            <origin
-                xyz="0 0 0"
-                rpy="0 0 0" />
-            <geometry>
-                <mesh
-                    filename="package://marvincar_description/meshes/front_handle_left.STL" />
+                    filename="package://marvin_description/meshes/front_handle_left.STL" />
+            </geometry>
+            <material
+                name="">
+                <color
+                    rgba="0.79216 0.81961 0.93333 1" />
+            </material>
+        </visual>
+        <collision>
+            <origin
+                xyz="0 0 0"
+                rpy="0 0 0" />
+            <geometry>
+                <mesh
+                    filename="package://marvin_description/meshes/front_handle_left.STL" />
             </geometry>
         </collision>
@@ -249,19 +249,19 @@
             <geometry>
                 <mesh
-                    filename="package://marvincar_description/meshes/front_wheel_left.STL" />
-            </geometry>
-            <material
-                name="">
-                <color
-                    rgba="0.79216 0.81961 0.93333 1" />
-            </material>
-        </visual>
-        <collision>
-            <origin
-                xyz="0 0 0"
-                rpy="0 0 0" />
-            <geometry>
-                <mesh
-                    filename="package://marvincar_description/meshes/front_wheel_left.STL" />
+                    filename="package://marvin_description/meshes/front_wheel_left.STL" />
+            </geometry>
+            <material
+                name="">
+                <color
+                    rgba="0.79216 0.81961 0.93333 1" />
+            </material>
+        </visual>
+        <collision>
+            <origin
+                xyz="0 0 0"
+                rpy="0 0 0" />
+            <geometry>
+                <mesh
+                    filename="package://marvin_description/meshes/front_wheel_left.STL" />
             </geometry>
         </collision>
@@ -307,19 +307,19 @@
             <geometry>
                 <mesh
-                    filename="package://marvincar_description/meshes/front_handle_right.STL" />
-            </geometry>
-            <material
-                name="">
-                <color
-                    rgba="0.79216 0.81961 0.93333 1" />
-            </material>
-        </visual>
-        <collision>
-            <origin
-                xyz="0 0 0"
-                rpy="0 0 0" />
-            <geometry>
-                <mesh
-                    filename="package://marvincar_description/meshes/front_handle_right.STL" />
+                    filename="package://marvin_description/meshes/front_handle_right.STL" />
+            </geometry>
+            <material
+                name="">
+                <color
+                    rgba="0.79216 0.81961 0.93333 1" />
+            </material>
+        </visual>
+        <collision>
+            <origin
+                xyz="0 0 0"
+                rpy="0 0 0" />
+            <geometry>
+                <mesh
+                    filename="package://marvin_description/meshes/front_handle_right.STL" />
             </geometry>
         </collision>
@@ -367,19 +367,19 @@
             <geometry>
                 <mesh
-                    filename="package://marvincar_description/meshes/front_wheel_right.STL" />
-            </geometry>
-            <material
-                name="">
-                <color
-                    rgba="0.79216 0.81961 0.93333 1" />
-            </material>
-        </visual>
-        <collision>
-            <origin
-                xyz="0 0 0"
-                rpy="0 0 0" />
-            <geometry>
-                <mesh
-                    filename="package://marvincar_description/meshes/front_wheel_right.STL" />
+                    filename="package://marvin_description/meshes/front_wheel_right.STL" />
+            </geometry>
+            <material
+                name="">
+                <color
+                    rgba="0.79216 0.81961 0.93333 1" />
+            </material>
+        </visual>
+        <collision>
+            <origin
+                xyz="0 0 0"
+                rpy="0 0 0" />
+            <geometry>
+                <mesh
+                    filename="package://marvin_description/meshes/front_wheel_right.STL" />
             </geometry>
         </collision>
