Commit message: fsdfdsf

File: marvin_sim_ws/src/marvin_description/urdf/marvin.urdf.xacro (robot description, xacro)
@@ -408,5 +408,5 @@
         <parent link="base_footprint" />
         <child link="base_link" />
-        <origin xyz="0 0 0" rpy="0 0 0" />
+        <origin xyz="0 0 0.05" rpy="0 0 0" />
     </joint>
     <gazebo reference="base_link">

File: marvin_sim_ws/src/marvin_description/urdf/sensors/camera_depth.xacro (robot description, xacro)
@@ -3,5 +3,5 @@
     <xacro:property name="M_PI" value="3.1415926535897931" />
     <joint name="joint_camera_depth" type="fixed">
-        <origin xyz="0.055 0 0.09" rpy="0 0 0" />
+        <origin xyz="0.055 0 0.11" rpy="0 0 0" />
         <parent link="base_link" />
         <child link="camera_depth" />

File: marvin_sim_ws/src/marvin_description/urdf/sensors/camera_left.xacro (robot description, xacro)
@@ -2,5 +2,5 @@
 <robot xmlns:xacro="http://ros.org/wiki/xacro">
     <joint name="joint_camera_left" type="fixed">
-        <origin xyz="-0.005 0.047832 0.095" rpy="0 0 ${pi/2}" />
+        <origin xyz="-0.005 0.047832 0.115" rpy="0 0 ${pi/2}" />
         <parent link="base_link" />
         <child link="camera_left" />

File: marvin_sim_ws/src/marvin_description/urdf/sensors/camera_right.xacro (robot description, xacro)
@@ -2,5 +2,5 @@
 <robot xmlns:xacro="http://ros.org/wiki/xacro">
     <joint name="joint_camera_right" type="fixed">
-        <origin xyz="-0.005 -0.047832 0.095" rpy="0 0 ${-pi/2}" />
+        <origin xyz="-0.005 -0.047832 0.115" rpy="0 0 ${-pi/2}" />
         <parent link="base_link" />
         <child link="camera_right" />

File: marvin_sim_ws/src/marvin_description/urdf/sensors/lidar.xacro (robot description, xacro)
@@ -49,5 +49,5 @@
         <joint name="${frame_id}_to_base_link" type="fixed">
             <origin
-                xyz="0 0 0.14"
+                xyz="0 0 0.158"
                 rpy="0 0 0" />
             <parent link="base_link" />

File: marvin_ws/src/marvincar_description/marvincar_description/urdf/sensors/camera_left.xacro (robot description, xacro)
@@ -2,5 +2,5 @@
 <robot xmlns:xacro="http://ros.org/wiki/xacro">
     <joint name="joint_camera_left" type="fixed">
-        <origin xyz="-0.005 0.047832 0.11" rpy="0 0 ${pi/2}" />
+        <origin xyz="-0.005 0.047832 0.115" rpy="0 0 ${pi/2}" />
         <parent link="base_link" />
         <child link="camera_left" />

File: marvin_ws/src/marvincar_description/marvincar_description/urdf/sensors/camera_right.xacro (robot description, xacro)
@@ -2,5 +2,5 @@
 <robot xmlns:xacro="http://ros.org/wiki/xacro">
     <joint name="joint_camera_right" type="fixed">
-        <origin xyz="-0.005 -0.047832 0.11" rpy="0 0 ${-pi/2}" />
+        <origin xyz="-0.005 -0.047832 0.115" rpy="0 0 ${-pi/2}" />
         <parent link="base_link" />
         <child link="camera_right" />
